File: electronics/plotting_robot.kicad_pcb (KiCad board)
At the start: 2 copper layers, 15 parts, among them Q2 BSS138, U2 ULN2003ADR, U4 ULN2003ADR

Commit message: Initial garbage layout
Parts:
- added J1: B5B-XH-A(LF)(SN), Connector_JST:JST_EH_B5B-EH-A_1x05_P2.50mm_Vertical, F.Cu at (191.5, 111.5)
- added J2: B5B-XH-A(LF)(SN), Connector_JST:JST_EH_B5B-EH-A_1x05_P2.50mm_Vertical, F.Cu at (129.0, 121.5)
- added J3: ~, Connector_PinHeader_2.54mm:PinHeader_1x03_P2.54mm_Vertical, F.Cu at (191.0, 103.0)
- added J4: Barrel_Jack_Switch, Library:DC-005, F.Cu at (181.0, 127.2)
- added J5: Conn_01x02_Pin, Connector_PinHeader_2.54mm:PinHeader_1x02_P2.54mm_Vertical, F.Cu at (173.0, 124.5)
- added U1: ~, Library:esp32_c3_oled, F.Cu at (156.2, 114.1)
- moved C1 50.7 mm to (172.0, 119.5), turned to -90 degrees
- moved C4 45.5 mm to (169.5, 119.0), turned to -90 degrees
- moved C2 45.1 mm to (185.0, 109.0), turned to 90 degrees
- moved C3 44.0 mm to (182.5, 109.5), turned to 90 degrees
- moved C5 39.8 mm to (172.0, 114.5), turned to -90 degrees
- moved C6 38.6 mm to (169.5, 115.0), turned to -90 degrees
- moved C10 37.2 mm to (136.5, 112.0), turned to 90 degrees
- moved U2 37.2 mm to (139.2, 119.6), turned to 90 degrees
- moved C7 34.7 mm to (185.5, 99.0), turned to 90 degrees
- moved C8 33.1 mm to (188.0, 99.0), turned to 90 degrees
- moved C9 31.3 mm to (139.0, 111.5), turned to 90 degrees
- moved U4 23.8 mm to (174.7, 106.8)
- moved R2 23.6 mm to (177.5, 98.0), turned to 180 degrees
- moved R1 17.9 mm to (169.5, 98.5), turned to -90 degrees
- moved Q2 16.5 mm to (173.1, 98.5)
Connections:
- C10 pad 1: +5V -> +5VP
- C2 pad 1: +5V -> +5VP
- C3 pad 1: +5V -> +5VP
- C7 pad 1: +5V -> +5VP
- C8 pad 1: +5V -> +5VP
- C9 pad 1: +5V -> +5VP
- U2 pad 9: +5V -> +5VP
- U4 pad 9: +5V -> +5VP
Routing:
- net +5VP: track 0.00 -> 133.4 mm, vias 0 -> 1
- net GND: track 0.00 -> 124.1 mm, vias 0 -> 3
- net +3V3: track 0.00 -> 39.7 mm, vias 0 -> 2
- net /M2C4: track 0.00 -> 26.1 mm, vias 0 -> 2
- net /M2C3: track 0.00 -> 25.6 mm, vias 0 -> 2
- net /M1C4: track 0.00 -> 25.2 mm
- net /M1C3: track 0.00 -> 25.1 mm
- net +5V: track 0.00 -> 24.7 mm, vias 0 -> 2
- net Net-(J1-COIL4): track 0.00 -> 23.3 mm
- net Net-(J1-COIL3): track 0.00 -> 22.5 mm
- net Net-(J1-COIL2): track 0.00 -> 21.1 mm
- net Net-(J1-COIL1): track 0.00 -> 20.0 mm
- net Net-(J3-SIG): track 0.00 -> 19.3 mm
- net /M1C2: track 0.00 -> 13.5 mm
- net /M2C1: track 0.00 -> 13.2 mm, vias 0 -> 1
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Other:
- board outline added: 68.1 x 32.5 mm

Commit message: Trying to get all JLPCB components
Parts:
- added Q1: BSS138W, PCM_JLCPCB:Q_SOT-323, F.Cu at (175.7, 95.1)
